File: Gesture Sensor.sch (KiCad schematic (older format))
At the start: 18 parts, among them J1 Conn_01x06_Male, J2 SM04B-SRSS-TB(LF)(SN), J3 SM04B-SRSS-TB(LF)(SN), U1 APDS-9960

Commit message: Fixed schematic issue with Mosfet
Parts:
- H1, H2, H3, H4: footprint MountingHole:MountingHole_2.5mm_Pad -> MountingHole:MountingHole_2.2mm_M2_ISO14580_Pad
- J1: value Conn_01x06_Male -> Conn_01x05_Male; footprint Connector_PinHeader_2.54mm:PinHeader_1x06_P2.54mm_Vertical -> Connector_PinHeader_2.54mm:PinHeader_1x05_P2.54mm_Vertical; symbol Connector:Conn_01x06_Male -> Connector:Conn_01x05_Male
- J2, J3: footprint JST_SM04B-SRSS-TB(LF)(SN) -> SM04B-SRSS-TB_LF__SN_:JST_SM04B-SRSS-TB(LF)(SN)
Connections:
- net VL is gone; now on net GND: J1.1 (Pin_1)
- net +3V3: now also JP1.2 (B); no longer JP1.1 (A)
- net GND: no longer J1.3 (Pin_3)
- net INT: now also J1.5 (Pin_5); no longer J1.6 (Pin_6)
- net SCL: now also J1.4 (Pin_4); no longer J1.5 (Pin_5)
- net SDA: now also J1.3 (Pin_3); no longer J1.4 (Pin_4)
- net at R2.1, R3.1: now also JP1.1 (A); no longer JP1.2 (B)
- net LDR: now reaches U1.3 (LDR), U1.4 (LEDK)
- net VDD: now reaches C3.1, R4.1, U1.8 (VDD)
Other:
- moved on the sheet: C1, C2, C3, JP1, R4
